Commit message: connecting UI buttons to intents for ros4hri compliance -wip

File: vulcanexus_ws/src/robin_core_bringup/urdf/scene_macro.xacro (robot description, xacro)
@@ -5,4 +5,5 @@
   <link name="weld_table">
     <visual>
+      <origin xyz="0 0 0" rpy="0 0 0"/>
       <geometry>
         <mesh filename="package://robin_core_bringup/meshes/welding_table/visual/WeldingTable.stl"/>

File: vulcanexus_ws/src/robin_core_bringup/urdf/sim_ur_fronius_garmo.urdf.xacro (robot description, xacro)
@@ -7,5 +7,5 @@
     <xacro:arg name="garmo_origin_rpy" default="${pi} 0 -${pi/2}"/>
     <xacro:arg name="welding_table_origin_xyz" default="-1.096 0.076 -0.193"/>
-    <xacro:arg name="welding_table_origin_rpy" default="0 0 ${pi/2}"/>
+    <xacro:arg name="welding_table_origin_rpy" default="0 0 0"/>
     <xacro:arg name="robot_platform_origin_xyz" default="0.25 0.4 -0.5"/>
     <xacro:arg name="robot_platform_origin_rpy" default="0 0 0"/>
@@ -21,5 +21,5 @@
     <!-- Add Fronius weld torch -->
     <xacro:fronius_weld_torch parent="tool0">
-        <origin xyz="0 0 0" rpy="0 0 0"/>
+        <origin xyz="0 0 0" rpy="0 0 ${pi}"/>
     </xacro:fronius_weld_torch>
     <!-- Add Garmo Garline laser sensor -->

File: vulcanexus_ws/src/robin_core_bringup/urdf/ur_fronius_garmo.urdf.xacro (robot description, xacro)
@@ -21,5 +21,5 @@
     <!-- Add Fronius weld torch -->
     <xacro:fronius_weld_torch parent="tool0">
-        <origin xyz="0 0 0" rpy="0 0 0"/>
+        <origin xyz="0 0 0" rpy="0 0 ${pi}"/>
     </xacro:fronius_weld_torch>
     <!-- Add Garmo Garline laser sensor -->

File: vulcanexus_ws/src/robin_hardware_fronius/urdf/fronius_macro.xacro (robot description, xacro)
@@ -5,4 +5,5 @@
         <link name="weld_torch">
         <visual>
+            <origin xyz="0 0 0" rpy="0 0 0"/>
             <geometry>
                 <mesh filename="package://robin_hardware_fronius/meshes/weld_torch/visual/weld_torch.obj"/>

File: vulcanexus_ws/src/robin_hardware_garmo/urdf/garmo_garline_macro.xacro (robot description, xacro)
@@ -12,4 +12,5 @@
     <link name="garmo_sensor_link">
       <visual>
+        <origin xyz="0 0 0" rpy="${-pi/2} 0 0"/>
         <!-- Use garmo_garline visual mesh -->
         <geometry>
