Commit message: adding test simulation of welding robot

File: vulcanexus_ws/src/robin_hardware_garmo/urdf/garmo_garline_macro.xacro (robot description, xacro)
@@ -12,5 +12,5 @@
     <link name="garmo_sensor_link">
       <visual>
-        <origin xyz="0 0 0" rpy="${-pi/2} 0 0"/>
+        <origin xyz="0 0 0" rpy="0 0 0"/>
         <!-- Use garmo_garline visual mesh -->
         <geometry>
