Commit message: ros4hri docs first draft + vulcanexus ws refactor to ROBIN implementation

File: vulcanexus_ws/src/robin_hardware_fronius/urdf/fronius_macro.xacro (robot description, xacro)
@@ -2,8 +2,7 @@
 <robot xmlns:xacro="http://www.ros.org/wiki/xacro" name="fronius">
   <!-- Define Fronius macro -->
-    <xacro:macro name="fronius_weld_torch" params="parent *origin">
+    <xacro:macro name="fronius_weld_torch" params="parent sim:=false ctwd:=0.015 tip_x:=0.00 tip_y:=-0.095 tip_z:=0.63 tip_roll:=${-pi/6} tip_pitch:=0 tip_yaw:=0 *origin">
         <link name="weld_torch">
         <visual>
-            <origin xyz="0 0 0" rpy="0 0 0"/>
             <geometry>
                 <mesh filename="package://robin_hardware_fronius/meshes/weld_torch/visual/weld_torch.obj"/>
@@ -21,5 +20,6 @@
         </inertial>
         </link>
-        <link name="weld_torch_tip">
+        <!-- Contact tip: where the wire exits the torch nozzle (red sphere) -->
+        <link name="contact_tip">
         <visual>
             <geometry>
@@ -36,9 +36,59 @@
         </inertial>
         </link>
-        <joint name="weld_torch_tip_joint" type="fixed">
+        <joint name="contact_tip_joint" type="fixed">
         <parent link="weld_torch"/>
-        <child link="weld_torch_tip"/>
-        <origin xyz="0.00 -0.085 0.645" rpy="-${pi/6} 0 0"/>
+        <child link="contact_tip"/>
+        <!-- Contact tip position relative to torch mesh origin (configurable via xacro args) -->
+        <origin xyz="${tip_x} ${tip_y} ${tip_z}" rpy="${tip_roll} ${tip_pitch} ${tip_yaw}"/>
         </joint>
+        <!-- Wire tip (actual TCP) - offset from contact tip by CTWD along wire direction (local Z) -->
+        <link name="wire_tip">
+        <visual>
+            <!-- Wire cylinder: 1mm diameter, 50mm long, extending behind wire_tip -->
+            <origin xyz="0 0 -0.025" rpy="0 0 0"/>
+            <geometry>
+                <cylinder radius="0.0005" length="0.05"/>
+            </geometry>
+            <material name="wire_silver">
+                <color rgba="0.75 0.75 0.75 1"/>
+            </material>
+        </visual>
+        <!-- Keep existing small sphere at tip -->
+        <visual>
+            <geometry>
+                <sphere radius="0.002"/>
+            </geometry>
+            <material name="yellow">
+                <color rgba="1 1 0 1"/>
+            </material>
+        </visual>
+        <collision>
+            <geometry>
+                <sphere radius="0.003"/>
+            </geometry>
+        </collision>
+        <inertial>
+            <mass value="0.01"/>
+            <origin xyz="0 0 0" rpy="0 0 0"/>
+            <inertia ixx="0.000001" ixy="0" ixz="0" iyy="0.000001" iyz="0" izz="0.000001"/>
+        </inertial>
+        </link>
+        <joint name="wire_tip_joint" type="fixed">
+            <parent link="contact_tip"/>
+            <child link="wire_tip"/>
+            <origin xyz="0 0 ${ctwd}" rpy="0 0 0"/>
+        </joint>
+        <!-- Prevent Gazebo fixed-joint lumping so wire_tip survives as a link -->
+        <gazebo reference="wire_tip_joint">
+            <preserveFixedJoint>true</preserveFixedJoint>
+        </gazebo>
+        <!-- Load Gazebo bead deposition plugin in sim mode -->
+        <xacro:if value="${sim}">
+        <gazebo>
+            <plugin filename="robin_sim_plugin" name="robin_sim_gz::RobinSimPlugin">
+                <weld_active_topic>/robin/weld_active</weld_active_topic>
+            </plugin>
+        </gazebo>
+        </xacro:if>
         <joint name="weld_torch_joint" type="fixed">
         <parent link="${parent}"/>

File: vulcanexus_ws/src/robin_hardware_garmo/urdf/garmo_garline_macro.xacro (robot description, xacro)
@@ -8,9 +8,8 @@
   -->
   <xacro:macro name="garmo_laser_sensor"
-               params="parent *origin">
+              params="parent sim:=false *origin">
     <!-- Sensor link -->
     <link name="garmo_sensor_link">
       <visual>
-        <origin xyz="0 0 0" rpy="0 0 0"/>
         <!-- Use garmo_garline visual mesh -->
         <geometry>
@@ -43,4 +42,49 @@
       <child link="laser_frame"/>
     </joint>
+    <!-- Gazebo GPU lidar – simulates the laser line profiler (sim only) -->
+    <xacro:if value="${sim}">
+      <!-- Sim lidar origin: at sensor body, pitched to aim at surface -->
+      <link name="sim_lidar_frame"/>
+      <joint name="sim_lidar_joint" type="fixed">
+        <origin xyz="0 0 0" rpy="0 1.4246 0"/>
+        <parent link="garmo_sensor_link"/>
+        <child link="sim_lidar_frame"/>
+      </joint>
+      <gazebo reference="sim_lidar_frame">
+        <sensor name="garmo_lidar" type="gpu_lidar">
+          <update_rate>42</update_rate>
+          <topic>/garmo_laser</topic>
+          <gz_frame_id>sim_lidar_frame</gz_frame_id>
+          <lidar>
+            <scan>
+              <horizontal>
+                <samples>500</samples>
+                <resolution>1</resolution>
+                <min_angle>-0.0812</min_angle>
+                <max_angle>0.0812</max_angle>
+              </horizontal>
+              <vertical>
+                <samples>1</samples>
+                <resolution>1</resolution>
+                <min_angle>0</min_angle>
+                <max_angle>0</max_angle>
+              </vertical>
+            </scan>
+            <range>
+              <min>0.137</min>
+              <max>0.207</max>
+              <resolution>0.0001</resolution>
+            </range>
+            <noise>
+              <type>gaussian</type>
+              <mean>0.0</mean>
+              <stddev>0.00025</stddev>
+            </noise>
+          </lidar>
+          <always_on>true</always_on>
+          <visualize>true</visualize>
+        </sensor>
+      </gazebo>
+    </xacro:if>
   </xacro:macro>
   <!-- example usage:

File: vulcanexus_ws/src/robin_hardware_ur/urdf/ur.urdf.xacro (robot description, xacro)
@@ -8,9 +8,10 @@
   <!-- possible 'ur_type' values: ur3, ur3e, ur5, ur5e, ur7e, ur10, ur10e, ur12e, ur16e, ur15, ur20, ur30 -->
   <!-- the default value should raise an error in case this was called without defining the type -->
+  <xacro:arg name="name" default="ur10e"/>
   <xacro:arg name="ur_type" default="ur10e"/>
   <!-- parameters -->
   <xacro:arg name="tf_prefix" default="" />
   <xacro:arg name="joint_limit_params" default="$(find ur_description)/config/$(arg ur_type)/joint_limits.yaml"/>
-  <xacro:arg name="kinematics_params" default="$(find ur_description)/config/$(arg ur_type)/default_kinematics.yaml"/>
+  <xacro:arg name="kinematics_params" default="$(find robin_hardware_ur)/config/robot_kinematics.yaml"/>
   <xacro:arg name="physical_params" default="$(find ur_description)/config/$(arg ur_type)/physical_parameters.yaml"/>
   <xacro:arg name="visual_params" default="$(find ur_description)/config/$(arg ur_type)/visual_parameters.yaml"/>

File: vulcanexus_ws/src/robin_hardware_ur/urdf/ur_gz.urdf.xacro (robot description, xacro)
@@ -35,5 +35,4 @@
     safety_pos_margin="$(arg safety_pos_margin)"
     safety_k_position="$(arg safety_k_position)"
-    force_abs_paths="true"
     >
     <origin xyz="0 0 0" rpy="0 0 0" />          <!-- position robot in the world -->
@@ -54,4 +53,5 @@
     tf_prefix="$(arg tf_prefix)"
     transmission_hw_interface="$(arg transmission_hw_interface)"
+    initial_positions="${dict(shoulder_pan_joint=2.7636586735327953,shoulder_lift_joint=-1.6422938239997316,elbow_joint=1.7227086417208768,wrist_1_joint=-2.143056021236931,wrist_2_joint=-1.3849973318064979,wrist_3_joint=-0.3312051136751893)}"
   />
 </robot>

File: vulcanexus_ws/src/robin_moveit_config/srdf/ur_macro.srdf.xacro (robot description, xacro)
@@ -13,14 +13,14 @@
     <!-- Main planning group - using ur_manipulator for compatibility with standard UR configs -->
     <group name="ur_manipulator">
-      <chain base_link="base_link" tip_link="weld_torch_tip" />
+      <chain base_link="base_link" tip_link="wire_tip" />
     </group>
     <!--GROUP STATES - Purpose - Define a named state for a particular group, in terms of joint values. This is useful to define states like 'folded arms'-->
     <group_state name="home" group="ur_manipulator">
-      <joint name="shoulder_pan_joint" value="0" />
-      <joint name="shoulder_lift_joint" value="-1.5707" />
-      <joint name="elbow_joint" value="0" />
-      <joint name="wrist_1_joint" value="-1.5707" />
-      <joint name="wrist_2_joint" value="0" />
-      <joint name="wrist_3_joint" value="0" />
+      <joint name="shoulder_pan_joint" value="2.763658" />
+      <joint name="shoulder_lift_joint" value="-1.64229" />
+      <joint name="elbow_joint" value="1.7227086" />
+      <joint name="wrist_1_joint" value="-2.143056" />
+      <joint name="wrist_2_joint" value="-1.384997" />
+      <joint name="wrist_3_joint" value="-0.331205" />
     </group_state>
     <group_state name="up" group="ur_manipulator">
@@ -32,16 +32,8 @@
       <joint name="wrist_3_joint" value="0" />
     </group_state>
-    <group_state name="test_configuration" group="ur_manipulator">
-      <joint name="shoulder_pan_joint" value="1.54" />
-      <joint name="shoulder_lift_joint" value="-1.62" />
-      <joint name="elbow_joint" value="1.4" />
-      <joint name="wrist_1_joint" value="-1.2" />
-      <joint name="wrist_2_joint" value="-1.6" />
-      <joint name="wrist_3_joint" value="-0.11" />
-    </group_state>
-    <!--END EFFECTOR - Commented out since weld_torch_tip is part of the ur_manipulator chain -->
-    <!-- <end_effector name="weld_torch" parent_group="ur_manipulator" group="ur_manipulator" parent_link="weld_torch_tip" /> -->
+    <!--END EFFECTOR - Commented out since contact_tip is part of the ur_manipulator chain -->
+    <!-- <end_effector name="weld_torch" parent_group="ur_manipulator" group="ur_manipulator" parent_link="contact_tip" /> -->
     <!--VIRTUAL JOINT - Purpose - this element defines a virtual joint between a robot link and an external frame of reference (considered fixed with respect to the robot)-->
-    <!-- <virtual_joint name="world_joint" type="fixed" parent_frame="world" child_link="base_link" /> -->
+    <virtual_joint name="world_joint" type="fixed" parent_frame="world" child_link="base_link" />
     <!--DISABLE COLLISIONS - By default it is assumed that any link of the robot could potentially come into collision with any other link in the robot. This tag disables collision checking between a specified pair of links. -->
     <disable_collisions link1="base_link" link2="robot_platform" reason="Adjacent" />
@@ -62,4 +54,9 @@
     <disable_collisions link1="wrist_2_link" link2="weld_torch" reason="Never" />
     <disable_collisions link1="wrist_3_link" link2="weld_torch" reason="Adjacent" />
+    <disable_collisions link1="weld_torch" link2="contact_tip" reason="Adjacent" />
+    <disable_collisions link1="contact_tip" link2="wire_tip" reason="Adjacent" />
+    <disable_collisions link1="wire_tip" link2="weld_table" reason="Never" />
+    <disable_collisions link1="weld_torch" link2="weld_table" reason="Never" />
+    <disable_collisions link1="contact_tip" link2="weld_table" reason="Never" />
   </xacro:macro>
 </robot>
