Commit message: ros2 package adaptation for no-hardware demo

File: vulcanexus_ws/src/robin_description/urdf/fronius_macro.xacro (robot description, xacro)
@@ -2,14 +2,14 @@
 <robot xmlns:xacro="http://www.ros.org/wiki/xacro" name="fronius">
   <!-- Define Fronius macro -->
-    <xacro:macro name="fronius_weld_torch" params="parent sim:=false ctwd:=0.015 tip_x:=0.00 tip_y:=-0.095 tip_z:=0.63 tip_roll:=${-pi/6} tip_pitch:=0 tip_yaw:=0 *origin">
+    <xacro:macro name="fronius_weld_torch" params="parent ctwd:=0.015 tip_x:=0.00 tip_y:=-0.095 tip_z:=0.63 tip_roll:=${-pi/6} tip_pitch:=0 tip_yaw:=0 *origin">
         <link name="weld_torch">
         <visual>
             <geometry>
-                <mesh filename="package://robin_hardware_fronius/meshes/weld_torch/visual/weld_torch.obj"/>
+                <mesh filename="package://robin_description/meshes/weld_torch/visual/weld_torch.obj"/>
             </geometry>
         </visual>
         <collision>
             <geometry>
-                <mesh filename="package://robin_hardware_fronius/meshes/weld_torch/collision/weld_torch.stl"/>
+                <mesh filename="package://robin_description/meshes/weld_torch/collision/weld_torch.stl"/>
             </geometry>
         </collision>
@@ -79,16 +79,4 @@
             <origin xyz="0 0 ${ctwd}" rpy="0 0 0"/>
         </joint>
-        <!-- Prevent Gazebo fixed-joint lumping so wire_tip survives as a link -->
-        <gazebo reference="wire_tip_joint">
-            <preserveFixedJoint>true</preserveFixedJoint>
-        </gazebo>
-        <!-- Load Gazebo bead deposition plugin in sim mode -->
-        <xacro:if value="${sim}">
-        <gazebo>
-            <plugin filename="robin_sim_plugin" name="robin_sim_gz::RobinSimPlugin">
-                <weld_active_topic>/robin/weld_active</weld_active_topic>
-            </plugin>
-        </gazebo>
-        </xacro:if>
         <joint name="weld_torch_joint" type="fixed">
         <parent link="${parent}"/>

File: vulcanexus_ws/src/robin_description/urdf/garmo_garline_macro.xacro (robot description, xacro)
@@ -8,5 +8,5 @@
   -->
   <xacro:macro name="garmo_laser_sensor"
-              params="parent sim:=false *origin">
+              params="parent *origin">
     <!-- Sensor link -->
     <link name="garmo_sensor_link">
@@ -14,5 +14,5 @@
         <!-- Use garmo_garline visual mesh -->
         <geometry>
-          <mesh filename="package://robin_hardware_garmo/meshes/garmo_garline/garmo_garline_visual.obj"/>
+          <mesh filename="package://robin_description/meshes/garmo_garline/garmo_garline_visual.obj"/>
         </geometry>
       </visual>
@@ -20,5 +20,5 @@
         <!-- Use garmo_garline collision mesh -->
         <geometry>
-          <mesh filename="package://robin_hardware_garmo/meshes/garmo_garline/garmo_garline_collision.stl"/>
+          <mesh filename="package://robin_description/meshes/garmo_garline/garmo_garline_collision.stl"/>
         </geometry>
       </collision>
@@ -42,49 +42,4 @@
       <child link="laser_frame"/>
     </joint>
-    <!-- Gazebo GPU lidar – simulates the laser line profiler (sim only) -->
-    <xacro:if value="${sim}">
-      <!-- Sim lidar origin: at sensor body, pitched to aim at surface -->
-      <link name="sim_lidar_frame"/>
-      <joint name="sim_lidar_joint" type="fixed">
-        <origin xyz="0 0 0" rpy="0 1.4246 0"/>
-        <parent link="garmo_sensor_link"/>
-        <child link="sim_lidar_frame"/>
-      </joint>
-      <gazebo reference="sim_lidar_frame">
-        <sensor name="garmo_lidar" type="gpu_lidar">
-          <update_rate>42</update_rate>
-          <topic>/garmo_laser</topic>
-          <gz_frame_id>sim_lidar_frame</gz_frame_id>
-          <lidar>
-            <scan>
-              <horizontal>
-                <samples>500</samples>
-                <resolution>1</resolution>
-                <min_angle>-0.0812</min_angle>
-                <max_angle>0.0812</max_angle>
-              </horizontal>
-              <vertical>
-                <samples>1</samples>
-                <resolution>1</resolution>
-                <min_angle>0</min_angle>
-                <max_angle>0</max_angle>
-              </vertical>
-            </scan>
-            <range>
-              <min>0.137</min>
-              <max>0.207</max>
-              <resolution>0.0001</resolution>
-            </range>
-            <noise>
-              <type>gaussian</type>
-              <mean>0.0</mean>
-              <stddev>0.00025</stddev>
-            </noise>
-          </lidar>
-          <always_on>true</always_on>
-          <visualize>true</visualize>
-        </sensor>
-      </gazebo>
-    </xacro:if>
   </xacro:macro>
   <!-- example usage:

File: vulcanexus_ws/src/robin_description/urdf/robin_tools.xacro (robot description, xacro)
@@ -4,9 +4,8 @@
          Include this in any bringup URDF after the UR robot is defined. -->
     <!-- Component macros -->
-    <xacro:include filename="$(find robin_hardware_fronius)/urdf/fronius_macro.xacro"/>
-    <xacro:include filename="$(find robin_hardware_garmo)/urdf/garmo_garline_macro.xacro"/>
-    <xacro:include filename="$(find robin_bringup)/urdf/scene_macro.xacro"/>
+    <xacro:include filename="$(find robin_description)/urdf/fronius_macro.xacro"/>
+    <xacro:include filename="$(find robin_description)/urdf/garmo_garline_macro.xacro"/>
+    <xacro:include filename="$(find robin_description)/urdf/scene_macro.xacro"/>
     <!-- Fronius weld torch params -->
-    <xacro:arg name="sim" default="false"/>
     <xacro:arg name="ctwd" default="0.015"/>
     <xacro:arg name="tip_x" default="0.00"/>
@@ -28,10 +27,9 @@
         ctwd="$(arg ctwd)"
         tip_x="$(arg tip_x)" tip_y="$(arg tip_y)" tip_z="$(arg tip_z)"
-        tip_roll="$(arg tip_roll)" tip_pitch="$(arg tip_pitch)" tip_yaw="$(arg tip_yaw)"
-        sim="$(arg sim)">
+        tip_roll="$(arg tip_roll)" tip_pitch="$(arg tip_pitch)" tip_yaw="$(arg tip_yaw)">
         <origin xyz="0 0 0" rpy="0 0 0"/>
     </xacro:fronius_weld_torch>
     <!-- Garmo Garline laser sensor on contact tip -->
-        <xacro:garmo_laser_sensor parent="contact_tip" sim="$(arg sim)">
+        <xacro:garmo_laser_sensor parent="contact_tip">
         <origin xyz="$(arg garmo_origin_xyz)" rpy="$(arg garmo_origin_rpy)"/>
     </xacro:garmo_laser_sensor>

File: vulcanexus_ws/src/robin_description/urdf/scene_macro.xacro (robot description, xacro)
@@ -6,5 +6,5 @@
     <visual>
       <geometry>
-        <mesh filename="package://robin_bringup/meshes/welding_table/visual/WeldingTable.stl"/>
+        <mesh filename="package://robin_description/meshes/welding_table/visual/WeldingTable.stl"/>
       </geometry>
       <material name="table_material">
@@ -15,5 +15,5 @@
       <origin xyz="0 0 0" rpy="0 0 0"/>
       <geometry>
-        <mesh filename="package://robin_bringup/meshes/welding_table/collision/WeldingTable.stl"/>
+        <mesh filename="package://robin_description/meshes/welding_table/collision/WeldingTable.stl"/>
       </geometry>
     </collision>

File: vulcanexus_ws/src/robin_description/urdf/ur.urdf.xacro (robot description, xacro)
@@ -13,5 +13,5 @@
   <xacro:arg name="tf_prefix" default="" />
   <xacro:arg name="joint_limit_params" default="$(find ur_description)/config/$(arg ur_type)/joint_limits.yaml"/>
-  <xacro:arg name="kinematics_params" default="$(find robin_hardware_ur)/config/robot_kinematics.yaml"/>
+  <xacro:arg name="kinematics_params" default="$(find robin_description)/config/robot_kinematics.yaml"/>
   <xacro:arg name="physical_params" default="$(find ur_description)/config/$(arg ur_type)/physical_parameters.yaml"/>
   <xacro:arg name="visual_params" default="$(find ur_description)/config/$(arg ur_type)/visual_parameters.yaml"/>

File: vulcanexus_ws/src/robin_description/urdf/ur_fronius_garmo.urdf.xacro (robot description, xacro)
@@ -1,6 +1,6 @@
 <?xml version="1.0"?>
 <robot xmlns:xacro="http://www.ros.org/wiki/xacro" name="robin_robot">
-    <!-- Real robot: UR10e + Fronius torch + Garmo laser + scene -->
-    <xacro:include filename="$(find robin_hardware_ur)/urdf/ur.urdf.xacro"/>
-    <xacro:include filename="$(find robin_bringup)/urdf/robin_tools.xacro"/>
+    <!-- UR10e + Fronius torch + Garmo laser + scene (hardware-agnostic description) -->
+    <xacro:include filename="$(find robin_description)/urdf/ur.urdf.xacro"/>
+    <xacro:include filename="$(find robin_description)/urdf/robin_tools.xacro"/>
 </robot>
